Commit message: temp

File: src/arm/arm_rviz/urdf/arm.urdf (robot description, URDF)
Before this commit: robot eyeexplorer, 6 links, 5 joints
Joints:
- joint arm_joint1: axis 0 1 0 -> 0 0 1; origin xyz=0 0.1 1.95 rpy=0 0 0 -> xyz=0 0 0 rpy=0 0 0
- joint arm_joint2: origin xyz=0 0.1 0.9 rpy=0 0 0 -> xyz=0 0 0 rpy=0 0 0
- joint arm_joint3: origin xyz=0 0 0.975 rpy=0 0 0 -> xyz=0 0 0 rpy=0 0 0; type fixed -> continuous
- joint arm_joint4: axis 0 1 0 -> 0.707106781 0 0.707106781; type fixed -> continuous

Commit message: とりあえずRViz2にアームらしきものがなんとなく表示できた（urdf要変更）

File: src/arm/arm_rviz/urdf/arm.urdf (robot description, URDF)
Before this commit: robot eyeexplorer, 6 links, 5 joints
Links:
- added link arm_link6, mass 1e-5; collision box size=0.05 0.05 0.05; visual box size=0.05 0.05 0.05
Joints:
- added joint arm_joint5: type continuous, parent arm_link5, child arm_link6, origin xyz=0.03982 0 -0.02239 rpy=0 0 0, axis 0.707106781 0 0.707106781
- joint arm_joint4: origin xyz=0.05 0 0.9 rpy=0 0 0 -> xyz=0.03982 0 -0.02239 rpy=0 0 0

Commit message: RViz2でロボットアーム表示

File: src/arm/arm_rviz/urdf/arm.urdf (robot description, URDF)
Before this commit: robot eyeexplorer, 7 links, 6 joints
Joints:
- removed joint arm_fixed
- added joint arm_joint_horiz: type continuous, parent arm_link3, child arm_link4, origin xyz=0 0 -0.2 rpy=0 0 0, axis 0 1 0
- joint arm_joint1: child arm_link2 -> arm_link1; origin xyz=0 0 0 rpy=0 0 0 -> xyz=0.2 0 0 rpy=0 0 0; parent arm_link1 -> world
- joint arm_joint2: child arm_link3 -> arm_link2; origin xyz=0 0 0 rpy=0 0 0 -> xyz=0 0 0.028 rpy=0 0 0; parent arm_link2 -> arm_link1
- joint arm_joint3: child arm_link4 -> arm_link3; origin xyz=0 0 0 rpy=0 0 0 -> xyz=0.2 0 0 rpy=0 0 0; parent arm_link3 -> arm_link2
- joint arm_joint4: axis 0.707106781 0 0.707106781 -> 1 0 0
- joint arm_joint5: axis 0.707106781 0 0.707106781 -> 0 1 0; origin xyz=0.03982 0 -0.02239 rpy=0 0 0 -> xyz=0 0 0 rpy=0 0 0

Commit message: stereo パッケージ追加

File: src/arm/arm_rviz/urdf/arm.urdf (robot description, URDF)
Before this commit: robot eyeexplorer, 7 links, 6 joints
Joints:
- joint arm_joint5: origin xyz=0 0 0 rpy=0 0 0 -> xyz=0.04 0 0 rpy=0 0 0
