Commit message: 3号機用URDFの変更など

File: src/arm/arm_rviz/urdf/eyeexplorer_ver3.urdf (robot description, URDF)
Before this commit: robot eyeexplorer, 7 links, 6 joints
Links:
- removed link arm_link5
- added link alm_frame; visual box size=0.5 0.03 0.03
- added link arm_link50; visual box size=0.02 0.06 0.02
- added link arm_link51; visual box size=0.06 0.02 0.02
- added link base; visual box size=0.03 0.03 0.08
- added link encoder_link; visual box size=0.01 0.01 0.04
- added link encoder_link2; visual box size=0.005 0.005 0.04
- link arm_link1: mass 1 -> None; geometry visual box size=0.03 0.03 0.032
- link arm_link2: mass 1 -> None; geometry visual box size=0.2 0.03 0.03
- link arm_link3: mass 1 -> None; geometry visual box size=0.03 0.03 -0.2
- link arm_link4: mass 1e-5 -> None; geometry visual box size=0.0349 0.03 0.03
- link arm_link6: mass 1e-5 -> None; geometry visual box size=0.02 -0.06 0.02
Joints:
- added joint arm_joint_gimbal: type fixed, parent arm_link50, child arm_link51, origin xyz=0 0.06 0 rpy=0 0 0
- added joint base_plate: type fixed, parent alm_frame, child base, origin xyz=0.5 0 0 rpy=0 0 0
- added joint encoder_joint: type fixed, parent arm_link6, child encoder_link, origin xyz=0 -0.06 0 rpy=0 0 0
- added joint encoder_joint2: type fixed, parent encoder_link, child encoder_link2, origin xyz=0 0 0.04 rpy=0 0 0
- added joint frame_joint: type fixed, parent world, child alm_frame
- joint arm_joint1: origin xyz=0.5 0 0 rpy=0 0 0 -> xyz=0 0 0.08 rpy=0 0 0; parent world -> base
- joint arm_joint4: child arm_link5 -> arm_link50; origin xyz=0.05654 0 -0.00486 rpy=0 0 0 -> xyz=0.0349 0 0.0 rpy=0 0 0
- joint arm_joint5: origin xyz=0.094 0 0 rpy=0 0 0 -> xyz=0.06 0 0 rpy=0 0 0; parent arm_link5 -> arm_link51
- joint arm_joint_horiz: origin xyz=0 0 -0.2 rpy=0 0 0 -> xyz=0.03232 0 -0.18232 rpy=0 0 0
