Commit message: FKをURDFに任せる、pclのテストなど

File: src/arm/arm_rviz/urdf/eyeexplorer3_nooffset.urdf (robot description, URDF)
Before this commit: robot eyeexplorer3, 11 links, 10 joints
Links:
- added link endoscope_holder_link; visual box size=0.02 0.02 -0.04
- link endoscope_link: geometry visual box size=0.01 0.01 -0.04
Joints:
- added joint endoscope_holder: type fixed, parent arm_link6, child endoscope_holder_link, origin xyz=0 0.06 0 rpy=0 0 0
- joint endoscope_joint: origin xyz=0 0.06 0 rpy=0 0 0 -> xyz=0 0 -0.04 rpy=0 0 0; parent arm_link6 -> endoscope_holder_link
- joint endoscope_joint2: origin xyz=0 0 -0.08 rpy=0 0 0 -> xyz=0 0 -0.04 rpy=0 0 0
