Commit message: EyeExplorer Calibratorだいたい完成

File: src/arm/arm_rviz/urdf/eyeexplorer3_fixed2.urdf (robot description, URDF)
Before this commit: robot eyeexplorer3, 13 links, 12 joints
Links:
- link arm_link51: geometry visual box size=0.1074 0.02 0.02
- link arm_link_para2: geometry visual box size=0.054 0.0005 -0.019
- link endoscope_holder_link: geometry visual box size=0.02 0.02 -0.03
- link endoscope_link: geometry visual box size=0.01 0.01 -0.03
Joints:
- joint arm_joint4: origin xyz=0.0415 0.005 -0.019 rpy=0 0 0 -> xyz=0.054 0.005 -0.019 rpy=0 0 0
- joint arm_joint5: origin xyz=0.0949 0 0 rpy=0 0 0 -> xyz=0.1074 0 0 rpy=0 0 0
- joint endoscope_joint: origin xyz=0 0 -0.04 rpy=0 0 0 -> xyz=0 0 -0.03 rpy=0 0 0
- joint endoscope_joint2: origin xyz=0 0 -0.04 rpy=0 0 0 -> xyz=0 0 -0.03 rpy=0 0 0

Commit message: メモリリーク問題解決

File: src/arm/arm_rviz/urdf/eyeexplorer3_fixed2.urdf (robot description, URDF)
Before this commit: robot eyeexplorer3, 13 links, 12 joints
Links:
- link arm_link_para2: geometry visual box size=0.054 0.02 -0.019
Joints:
- joint arm_joint4: origin xyz=0.054 0.005 -0.019 rpy=0 0 0 -> xyz=0.054 0.0005 -0.019 rpy=0 0 0
