Commit message: 3号機用にアーム変更完了

File: src/arm/arm_rviz/urdf/eyeexplorer3.urdf (robot description, URDF)
Before this commit: robot eyeexplorer3, 12 links, 11 joints
Links:
- removed link encoder_link
- removed link encoder_link2
- added link endoscope; visual box size=0 0 0
- added link endoscope_link; visual box size=0.01 0.01 -0.045
- added link endoscope_link2; visual box size=0.005 0.005 -0.045
- link arm_link50: geometry visual box size=0.02 -0.06 0.02
- link arm_link6: geometry visual box size=0.02 0.06 0.02
Joints:
- removed joint encoder_joint
- removed joint encoder_joint2
- added joint endoscope_camera: type fixed, parent endoscope_link2, child endoscope, origin xyz=0 0 0 rpy=0 3.14 -3.14
- added joint endoscope_joint: type fixed, parent arm_link6, child endoscope_link, origin xyz=0 0.06 0 rpy=0 0 0
- added joint endoscope_joint2: type fixed, parent endoscope_link, child endoscope_link2, origin xyz=0 0 -0.0225 rpy=0 0 0
- joint arm_joint_gimbal: origin xyz=0 0.06 0 rpy=0 0 0 -> xyz=0 -0.06 0 rpy=0 0 0

Commit message: 二重定義禁止とtf削除によってfKノードを安定化

File: src/arm/arm_rviz/urdf/eyeexplorer3.urdf (robot description, URDF)
Before this commit: robot eyeexplorer3, 13 links, 12 joints
Joints:
- joint endoscope_camera: origin xyz=0 0 0 rpy=0 3.14 -3.14 -> xyz=0 0 0 rpy=0 3.14 0

Commit message: armディレクトリ内ファイル整理

File: src/arm/arm_rviz/urdf/eyeexplorer3.urdf (robot description, URDF)
Before this commit: robot eyeexplorer3, 13 links, 12 joints
Links:
- removed link alm_frame
- removed link arm_link3
- removed link arm_link4
- removed link base
- added link arm_link_para1; visual box size=0.03232 0.03 0.01768
- added link arm_link_para2; visual box size=0.054 0.02 -0.019
- added link endoscope_holder_link; visual box size=0.02 0.02 -0.03
- added link link_base; visual box size=0.009 0.01 0.032
- link arm_link1: geometry visual box size=0.2 0.03 0.03
- link arm_link2: geometry visual box size=0.03 0.03 -0.2
- link arm_link51: geometry visual box size=0.1074 0.02 0.02
- link endoscope_link: geometry visual box size=0.01 0.01 -0.03
- link endoscope_link2: geometry visual box size=0.005 0.005 -0.03
Joints:
- removed joint arm_joint_horiz
- removed joint base_plate
- removed joint frame_joint
- added joint arm_joint_horiz1: type continuous, parent arm_link1, child arm_link_para1, origin xyz=0.2 0 0 rpy=0 0 0, axis 0 1 0
- added joint arm_joint_horiz2: type continuous, parent arm_link2, child arm_link_para2, origin xyz=0 0 -0.2 rpy=0 0 0, axis 0 1 0
- added joint endoscope_holder: type fixed, parent arm_link6, child endoscope_holder_link, origin xyz=0 0.06 0 rpy=0 0 0
- joint arm_joint1: child arm_link1 -> link_base; origin xyz=0 0 0.08 rpy=0 0 0 -> xyz=0.0 0 0.0 rpy=0 0 0; parent base -> world
- joint arm_joint2: child arm_link2 -> arm_link1; parent arm_link1 -> link_base
- joint arm_joint3: child arm_link3 -> arm_link2; origin xyz=0.2 0 0 rpy=0 0 0 -> xyz=0.03232 0 0.01768 rpy=0 0 0; parent arm_link2 -> arm_link_para1
- joint arm_joint4: origin xyz=0.0349 0 0.0 rpy=0 0 0 -> xyz=0.054 0.0005 -0.019 rpy=0 0 0; parent arm_link4 -> arm_link_para2
- joint arm_joint5: origin xyz=0.06 0 0 rpy=0 0 0 -> xyz=0.1074 0 0 rpy=0 0 0
- joint endoscope_camera: origin xyz=0 0 0 rpy=0 3.14 0 -> xyz=0 0 -0.03 rpy=0 3.14 0
- joint endoscope_joint: origin xyz=0 0.06 0 rpy=0 0 0 -> xyz=0 0 -0.03 rpy=0 0 0; parent arm_link6 -> endoscope_holder_link
- joint endoscope_joint2: origin xyz=0 0 -0.0225 rpy=0 0 0 -> xyz=0 0 -0.03 rpy=0 0 0

Commit message: マーカーの位置修正

File: src/arm/arm_rviz/urdf/eyeexplorer3.urdf (robot description, URDF)
Before this commit: robot eyeexplorer3, 13 links, 12 joints
Links:
- link endoscope_link2: geometry visual box size=0.005 0.005 -0.035
- link link_base: geometry visual box size=0.019 0.01 0.022
Joints:
- joint arm_joint2: origin xyz=0.009 0 0.032 rpy=0 0 0 -> xyz=0.019 0 0.022 rpy=0 0 0
- joint endoscope_camera: origin xyz=0 0 -0.03 rpy=0 3.14 0 -> xyz=0 0 -0.035 rpy=0 3.14 0

Commit message: 内視鏡の色と大きさを変更

File: src/arm/arm_rviz/urdf/eyeexplorer3.urdf (robot description, URDF)
Before this commit: robot eyeexplorer3, 13 links, 12 joints
Links:
- link endoscope_link2: geometry visual box size=0.002 0.002 -0.035

File: src/arm/arm_rviz/urdf/eyeexplorer3_dif.urdf (robot description, URDF)
Before this commit: robot eyeexplorer3, 15 links, 14 joints
Links:
- link endoscope_link_dif1: geometry visual box size=0.002 0.002 -0.03

Commit message: Update URDF

File: src/arm/arm_rviz/urdf/eyeexplorer3.urdf (robot description, URDF)
Before this commit: robot eyeexplorer3, 13 links, 12 joints
Links:
- link endoscope_link2: geometry visual cylinder length=0.035 radius=0.001

File: src/arm/arm_rviz/urdf/eyeexplorer3_dif.urdf (robot description, URDF)
Before this commit: robot eyeexplorer3, 15 links, 14 joints
Links:
- link endoscope_link_dif1: geometry visual cylinder length=0.035 radius=0.001
Joints:
- joint endoscope_camera_dif: origin xyz=0 0.005179 -0.03 rpy=-0.02899 0 0 -> xyz=0 0.005179 -0.035 rpy=-0.02899 0 0

Commit message: アームの長さ微調整

File: src/arm/arm_rviz/urdf/eyeexplorer3.urdf (robot description, URDF)
Before this commit: robot eyeexplorer3, 13 links, 12 joints
Links:
- link endoscope_link: geometry visual box size=0.01 0.01 -0.032
- link endoscope_link2: geometry visual cylinder length=0.028 radius=0.001
Joints:
- joint endoscope_camera: origin xyz=0 0 -0.035 rpy=0 3.14 0 -> xyz=0 0 -0.028 rpy=0 3.14 0
- joint endoscope_joint2: origin xyz=0 0 -0.03 rpy=0 0 0 -> xyz=0 0 -0.032 rpy=0 0 0

Commit message: fix arm link param

File: src/arm/arm_rviz/urdf/eyeexplorer3.urdf (robot description, URDF)
Before this commit: robot eyeexplorer3, 13 links, 12 joints
Links:
- link arm_link51: geometry visual box size=0.075 0.02 0.02
- link arm_link_para1: geometry visual box size=0.03586 0.03 0.01414
- link arm_link_para2: geometry visual box size=0.0614 0.02 -0.019
- link link_base: geometry visual box size=0.009 0.01 0.032
Joints:
- joint arm_joint2: origin xyz=0.019 0 0.022 rpy=0 0 0 -> xyz=0.009 0 0.032 rpy=0 0 0
- joint arm_joint3: origin xyz=0.03232 0 0.01768 rpy=0 0 0 -> xyz=0.03586 0 0.01414 rpy=0 0 0
- joint arm_joint4: origin xyz=0.054 0.0005 -0.019 rpy=0 0 0 -> xyz=0.0614 0.0 -0.019 rpy=0 0 0
- joint arm_joint5: origin xyz=0.1074 0 0 rpy=0 0 0 -> xyz=0.075 0 0 rpy=0 0 0
